Commit message: fix some errors

File: description/drive_unit.xacro (robot description, xacro)
@@ -46,5 +46,5 @@
             <parent link="${prefix}_motorbox" />
             <child link="${prefix}_wheel" />
-            <origin rpy="${pi/2} 0.0 0.0" xyz="0.0 ${(motorwidth+wheelwidth)/2} 0.0" />
+            <origin rpy="${pi/2} 0.0 0.0" xyz="0.0 ${wheelwidth/2} 0.0" />
             <axis rpy="0.0 0.0 0.0" xyz="0.0 0.0 1" />
         </joint>

File: description/rcw0001_sensor.xacro (robot description, xacro)
@@ -21,5 +21,5 @@
         <link name="${prefix}_rcw0001">
             <visual>
-                <origin xyz="-${rcwlength*4/5} 0.0 ${rcwheight/2}" />
+                <origin xyz="-${rcwlength*2/5} 0.0 0.0" />
                 <geometry>
                     <box size="${rcwlength/5} ${rcwwidth} ${rcwheight}" />
@@ -28,12 +28,19 @@
             </visual>
             <visual>
-                <origin xyz="${rcwlength/5} ${rcwwidth/2} ${rcwheight/2}" />
+                <origin rpy="0.0 ${pi/2} 0.0" xyz="${rcwlength/10} ${rcwwidth/4} 0.0" />
                 <geometry>
-                    <cylinder radius="${rcwheight/4}" length="${rcwlength*4/5}" />
+                    <cylinder radius="${rcwheight/2.2}" length="${rcwlength*4/5}" />
+                </geometry>
+                <material name="rcw0001-sensors" />
+            </visual>
+            <visual>
+                <origin rpy="0.0 ${pi/2} 0.0" xyz="${rcwlength/10} -${rcwwidth/4} 0.0" />
+                <geometry>
+                    <cylinder radius="${rcwheight/2.2}" length="${rcwlength*4/5}" />
                 </geometry>
                 <material name="rcw0001-sensors" />
             </visual>
             <collision>
-                <origin xyz="0.0 0.0 ${rcwheight/2}" />
+                <origin xyz="0.0 0.0 0.0" />
                 <geometry>
                     <box size="${rcwlength} ${rcwwidth} ${rcwheight}" />
