Commit message: pan-tilt-cam added

File: description/chassis.xacro (robot description, xacro)
@@ -111,3 +111,10 @@
     <xacro:rcw0001_joint prefix="rear_right" base="body" rotateZ="${pi+pi/6}" moveX="-0.115" moveY="-0.055" moveZ="-${bodyheight/2}" />
     <xacro:rcw0001 prefix="rear_right" />
+    <!-- PAN-TILT CAMERA -->
+    <joint name="base_to_pan_tilt_cam" type="fixed">
+        <parent link="body" />
+        <child link="pan_tilt_cam_base" />
+        <origin xyz="0.058 0.0 ${bodyheight/2}" />
+    </joint>
+    <xacro:include filename="pan_tilt_cam.xacro" />
 </robot>

File: description/pi_box.xacro (robot description, xacro)
@@ -4,5 +4,5 @@
     <xacro:property name="pilength" value="0.088" />
     <xacro:property name="piwidth" value="0.056" />
-    <xacro:property name="piheight" value="0.028" />
+    <xacro:property name="piheight" value="0.040" />
     <material name="pi-box">
         <color rgba="1.0 0.5 0.5 1.0" />
