Commit message: adjust joint direction

File: description/pan_tilt_cam.xacro (robot description, xacro)
@@ -37,5 +37,5 @@
         <child link="vertical_arm" />
         <origin rpy="0.0 0.0 0.0" xyz="0.0 0.0 ${v_armlength/2}" />
-        <axis rpy="0.0 0.0 0.0" xyz="0.0 0.0 1" />
+        <axis rpy="0.0 0.0 0.0" xyz="0.0 0.0 -1" />
         <limit lower="${-pi/3}" upper="${pi/3}" velocity="100" effort="100"/>
     </joint>
