Commit message: first simulation

File: description/camera.xacro (robot description, xacro)
@@ -35,3 +35,6 @@
         </xacro:inertial_box>
     </link>
+    <gazebo reference="camera">
+        <material>Gazebo/Black</material>
+    </gazebo>
 </robot>

File: description/chassis.xacro (robot description, xacro)
@@ -69,18 +69,21 @@
         </xacro:inertial_box>
     </link>
+    <gazebo reference="body">
+        <material>Gazebo/White</material>
+    </gazebo>
      <!-- DRIVE_UNITS -->
      <xacro:include filename="drive_unit.xacro" />
      <!-- front left -->
      <xacro:drive_joint prefix="front_left" base="body" rotateX="0" rotateY="0" rotateZ="0" moveX="${(bodylength+trunklength)/4}" moveY="${bodywidth/2}" moveZ="-${bodyheight/2}" />
-     <xacro:drive_unit prefix="front_left" />
+     <xacro:drive_unit prefix="front_left" direction="1" />
      <!-- front right -->
      <xacro:drive_joint prefix="front_right" base="body" rotateX="${pi}" rotateY="0" rotateZ="0" moveX="${(bodylength+trunklength)/4}" moveY="-${bodywidth/2}" moveZ="-${bodyheight/2}" />
-     <xacro:drive_unit prefix="front_right" />
+     <xacro:drive_unit prefix="front_right" direction="-1" />
      <!-- rear left -->
      <xacro:drive_joint prefix="rear_left" base="body" rotateX="${pi}" rotateY="0" rotateZ="${pi}" moveX="-${(bodylength+trunklength)/4}" moveY="${bodywidth/2}" moveZ="-${bodyheight/2}" />
-     <xacro:drive_unit prefix="rear_left" />
+     <xacro:drive_unit prefix="rear_left" direction="1" />
      <!-- rear right -->
       <xacro:drive_joint prefix="rear_right" base="body" rotateX="0" rotateY="0" rotateZ="${pi}" moveX="-${(bodylength+trunklength)/4}" moveY="-${bodywidth/2}" moveZ="-${bodyheight/2}" />
-     <xacro:drive_unit prefix="rear_right" />
+     <xacro:drive_unit prefix="rear_right" direction="-1" />
     <!-- PI-BOX -->
     <joint name="pi_box_joint" type="fixed">

File: description/drive_unit.xacro (robot description, xacro)
@@ -24,5 +24,5 @@
     </xacro:macro>
     <!-- Macro for drive_unit including motor, gearbox, wheel -->
-    <xacro:macro name="drive_unit" params="prefix">
+    <xacro:macro name="drive_unit" params="prefix direction">
         <link name="${prefix}_motorbox">
             <visual>
@@ -43,9 +43,12 @@
         </xacro:inertial_box>
         </link>
+        <gazebo reference="${prefix}_motorbox">
+            <material>Gazebo/Yellow</material>
+        </gazebo>
         <joint name="${prefix}_wheel_joint" type="continuous">
             <parent link="${prefix}_motorbox" />
             <child link="${prefix}_wheel" />
-            <origin rpy="${pi/2} 0.0 0.0" xyz="0.0 ${wheelwidth/2} 0.0" />
-            <axis rpy="0.0 0.0 0.0" xyz="0.0 0.0 1" />
+            <origin rpy="${-pi/2} 0.0 0.0" xyz="0.0 ${wheelwidth/2} 0.0" />
+            <axis rpy="0.0 0.0 0.0" xyz="0.0 0.0 ${direction}" />
         </joint>
         <link name="${prefix}_wheel">
@@ -65,4 +68,18 @@
             </xacro:inertial_cylinder>
         </link>
+        <gazebo reference="${prefix}_wheel">
+            <material>Gazebo/Black</material>
+            <mu1 value="0.5"/>
+            <mu2 value="0.5"/>
+            <kp value="1000000.0"/>
+            <kd value="1.0"/>
+<!--
+            <mu  value="0.1"/>
+            <slip  value="1.0" />
+            <slip1 value="1.0" />
+            <slip2 value="1.0" />
+            <fdir1 value="1 1 0"/>
+-->
+        </gazebo>
     </xacro:macro>
 </robot>

File: description/nodebot1.urdf.xacro (robot description, xacro)
@@ -7,3 +7,5 @@
     <!-- CHASSIS -->
     <xacro:include filename="chassis.xacro" />
+    <!-- Controls for Simulation with Gazebo -->
+    <xacro:include filename="gazebo_control.xacro" />
 </robot>

File: description/pan_tilt_cam.xacro (robot description, xacro)
@@ -33,4 +33,7 @@
         </xacro:inertial_box>
     </link>
+    <gazebo reference="pan_tilt_cam_base">
+        <material>Gazebo/Black</material>
+    </gazebo>
     <joint name="vertical_arm_joint" type="revolute">
         <parent link="pan_tilt_cam_base" />
@@ -56,4 +59,7 @@
         </xacro:inertial_cylinder>
     </link>
+    <gazebo reference="vertical_arm">
+        <material>Gazebo/Black</material>
+    </gazebo>
     <joint name="horizontal_arm_joint" type="fixed">
         <parent link="vertical_arm" />
@@ -79,4 +85,7 @@
         </xacro:inertial_box>
     </link>
+    <gazebo reference="horizontal_arm">
+        <material>Gazebo/Black</material>
+    </gazebo>
     <joint name="cam_plate_joint" type="revolute">
         <parent link="horizontal_arm" />
@@ -104,4 +113,7 @@
         </xacro:inertial_box>
     </link>
+    <gazebo reference="cam_plate">
+        <material>Gazebo/Black</material>
+    </gazebo>
     <joint name="camera_joint" type="fixed">
         <parent link="cam_plate" />

File: description/pi_box.xacro (robot description, xacro)
@@ -26,3 +26,6 @@
         </xacro:inertial_box>
     </link>
+    <gazebo reference="pi_box">
+        <material>Gazebo/Blue</material>
+    </gazebo>
 </robot>

File: description/rcw0001_sensor.xacro (robot description, xacro)
@@ -51,4 +51,7 @@
             </xacro:inertial_box>
         </link>
+        <gazebo reference="${prefix}_rcw0001">
+            <material>Gazebo/Green</material>
+        </gazebo>
     </xacro:macro>
 </robot>

File: description/vltg_box.xacro (robot description, xacro)
@@ -26,3 +26,6 @@
         </xacro:inertial_box>
     </link>
+    <gazebo reference="vltg_box">
+        <material>Gazebo/Blue</material>
+    </gazebo>
 </robot>

Commit message: basic cam arm physics

File: description/camera.xacro (robot description, xacro)
@@ -36,5 +36,5 @@
     </link>
     <gazebo reference="camera">
-        <material>Gazebo/Black</material>
+        <material>Gazebo/Orange</material>
     </gazebo>
 </robot>

File: description/drive_unit.xacro (robot description, xacro)
@@ -72,8 +72,8 @@
             <mu1 value="0.5"/>
             <mu2 value="0.5"/>
+<!--
+            <mu  value="0.5"/>
             <kp value="1000000.0"/>
             <kd value="1.0"/>
-<!--
-            <mu  value="0.1"/>
             <slip  value="1.0" />
             <slip1 value="1.0" />

File: description/gazebo_control.xacro (robot description, xacro)
@@ -25,4 +25,12 @@
             <robot_base_frame>base_link</robot_base_frame>
         </plugin>
+        <plugin name="gazebo_ros_joint_state_publisher" filename="libgazebo_ros_joint_state_publisher.so">
+            <update_rate>20</update_rate>
+            <joint_name>cam_plate_joint</joint_name>
+            <joint_name>vertical_arm_joint</joint_name>
+        </plugin>
+        <plugin name="gazebo_ros_joint_pose_trajectory" filename="libgazebo_ros_joint_pose_trajectory.so">
+            <update_rate>20</update_rate>
+        </plugin>
     </gazebo>
 </robot>

File: description/pan_tilt_cam.xacro (robot description, xacro)
@@ -41,5 +41,6 @@
         <origin rpy="0.0 0.0 0.0" xyz="0.0 0.0 ${v_armlength/2}" />
         <axis rpy="0.0 0.0 0.0" xyz="0.0 0.0 -1" />
-        <limit lower="${-pi/3}" upper="${pi/3}" velocity="100" effort="100"/>
+        <limit lower="${-pi/3}" upper="${pi/3}" velocity="100" effort="100" />
+        <dynamics damping="1.0" friction="1.0" />
     </joint>
     <link name="vertical_arm">
@@ -93,5 +94,6 @@
         <origin rpy="0.0 0.0 0.0" xyz="${h_armlength/2} 0.0 0.0" />
         <axis rpy="0.0 0.0 0.0" xyz="0.0 -1 0.0" />
-        <limit lower="${-pi/12}" upper="${5*pi/12}" velocity="100" effort="100"/>
+        <limit lower="${-pi/12}" upper="${5*pi/12}" velocity="100" effort="100" />
+        <dynamics damping="1.0" friction="1.0" />
     </joint>
     <link name="cam_plate">
